File: 1.0/1.0.kicad_pcb (KiCad board)
At the start: 4 copper layers, 120 x 80 mm, 151 parts, among them IC1 GD25Q16CWIGR, IC2 ATSAMD21G18A-MUT, J1 header_01x04, J2 USB_A, J3 header_01x04, J4 header_01x04, J5 header_01x04, J6 header_01x04, J7 uSDCard, P1 CONN_1, P2 CONN_1, Q1 BC847, Q10 PMOS_SGD, Q11 PMOS_SGD, Q12 PMOS_SGD, Q2 BC847, Q3 PMOS_SGD, Q4 PMOS_SGD, Q5 PMOS_SGD, Q6 PMOS_SGD, Q7 BC847, Q8 BC847, Q9 PMOS_SGD, SW1 SW_Push, U1 ARM-SWD-10, U10 LM1085-3.0, U11 LM1085-3.0, U12 LM1085-3.0, U13 PCT2075, U14 PCT2075, U15 XT90PW-M, U16 XT90PW-M, U17 XT90PW-M, U18 XT90PW-M, U19 XT90PW-M, U2 ACS781, U20 XT90PW-M, U21 XT90PW-M, U22 XT90PW-M, U23 XT90PW-M, U24 XT90PW-M, U25 XT90PW-M, U3 ACS781, U4 MPM3610, U5 MPM3610, U6 MPM3610, U7 LM1085-5.0, U8 LM1085-5.0, U9 LM1085-5.0

Commit message: updates
Parts:
- added TP10: TEST, 0_misc:test_point_2mm_square, F.Cu at (136.4, 138.3)
- added TP11: TEST, 0_misc:test_point_2mm_square, F.Cu at (130.4, 138.3)
- added TP12: TEST, 0_misc:test_point_2mm_square, F.Cu at (136.4, 132.3)
- added TP13: TEST, 0_misc:test_point_2mm_square, F.Cu at (130.4, 135.3)
- added TP2: TEST, 0_misc:test_point_2mm_square, F.Cu at (139.4, 132.3)
- added TP3: TEST, 0_misc:test_point_2mm_square, F.Cu at (133.4, 135.3)
- added TP4: TEST, 0_misc:test_point_2mm_square, F.Cu at (139.4, 135.3)
- added TP5: TEST, 0_misc:test_point_2mm_square, F.Cu at (136.4, 135.3)
- added TP6: TEST, 0_misc:test_point_2mm_square, F.Cu at (130.4, 132.3)
- added TP7: TEST, 0_misc:test_point_2mm_square, F.Cu at (133.4, 138.3)
- added TP8: TEST, 0_misc:test_point_2mm_square, F.Cu at (133.4, 132.3)
- added TP9: TEST, 0_misc:test_point_2mm_square, F.Cu at (142.4, 132.3)
- C11, R29: moved to F.Cu
- NT1: footprint 0_NetTie:NetTie-4_SMD_Pad2.0mm -> 0_NetTie:NetTie-2_SMD_Pad2.0mm
- moved U4 195.9 mm to (177.9, 146.4)
- moved R33 195.9 mm to (175.2, 146.9)
- moved R32 195.9 mm to (175.2, 144.0)
- moved R29 194.3 mm to (176.8, 141.9), turned to -90 degrees
- moved C11 191.1 mm to (179.2, 142.4)
- moved C14 174.1 mm to (180.8, 147.2), turned to 90 degrees
- moved U19 147.4 mm to (208.7, 194.4)
- moved D5 104.4 mm to (198.1, 88.7)
- moved R15 104.4 mm to (195.9, 89.5)
- moved C9 57.1 mm to (260.8, 108.7)
- moved C6 41.5 mm to (269.6, 164.6)
- moved D4 21.7 mm to (182.3, 103.3), turned to 180 degrees
- moved R9 19.0 mm to (181.6, 105.5), turned to 90 degrees
- moved C5 12.4 mm to (202.8, 173.1)
- moved R5 10.2 mm to (181.7, 161.7)
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Connections:
- U5 pad 14: GNDD -> GND
- U5 pad 3: GNDD -> GND
- U6 pad 14: GNDD -> GND
- U6 pad 3: GNDD -> GND
Routing:
- net +3V3: vias 0 -> 1
- added copper zone on In2.Cu, net +3V3

Commit message: updates
Parts:
- removed TP2: TEST, 0_misc:test_point_2mm_square
- added D11: LED, 2_Passives_Resistors_SMD_IPC:R_1608_603_B, F.Cu at (219.9, 115.7)
- added D6: LED, 2_Passives_Resistors_SMD_IPC:R_1608_603_B, F.Cu at (219.3, 164.8)
- added J10: header_01x03, 5_Connectors_Molex:MegaF_RAH_Single_3x5.7mm, F.Cu at (306.7, 122.4)
- added J11: header_01x03, 5_Connectors_Molex:MegaF_RAH_Single_3x5.7mm, F.Cu at (327.6, 122.4)
- added J12: header_01x03, 5_Connectors_Molex:MegaF_RAH_Single_3x5.7mm, F.Cu at (327.7, 158.0)
- added J13: header_01x03, 5_Connectors_Molex:MegaF_RAH_Single_3x5.7mm, F.Cu at (264.6, 158.0)
- added J14: header_01x03, 5_Connectors_Molex:MegaF_RAH_Single_3x5.7mm, F.Cu at (285.7, 157.9)
- added J15: header_01x03, 5_Connectors_Molex:MegaF_RAH_Single_3x5.7mm, F.Cu at (306.5, 157.9)
- added J8: header_01x03, 5_Connectors_Molex:MegaF_RAH_Single_3x5.7mm, F.Cu at (264.6, 122.7)
- added J9: header_01x03, 5_Connectors_Molex:MegaF_RAH_Single_3x5.7mm, F.Cu at (285.8, 122.7)
- added R16: 300, 2_Passives_Resistors_SMD_IPC:R_1608_603_B, F.Cu at (213.7, 163.5)
- added R58: 300, 2_Passives_Resistors_SMD_IPC:R_1608_603_B, F.Cu at (215.1, 163.5)
- added R59: 300, 2_Passives_Resistors_SMD_IPC:R_1608_603_B, F.Cu at (216.5, 163.5)
- added R60: 300, 2_Passives_Resistors_SMD_IPC:R_1608_603_B, F.Cu at (222.8, 117.1)
- added R61: 300, 2_Passives_Resistors_SMD_IPC:R_1608_603_B, F.Cu at (222.8, 115.7)
- added TP14: TEST, 0_misc:test_point_2mm_square, B.Cu at (167.5, 146.4)
- added TP15: TEST, 0_misc:test_point_2mm_square, B.Cu at (165.1, 148.8)
- added TP16: TEST, 0_misc:test_point_2mm_square, B.Cu at (187.5, 140.0)
- added U26: ESC, hot_swap_footprints:esc, B.Cu at (264.6, 120.1)
- added U27: ESC, hot_swap_footprints:esc, B.Cu at (285.6, 120.2)
- added U28: ESC, hot_swap_footprints:esc, B.Cu at (306.6, 120.2)
- added U29: ESC, hot_swap_footprints:esc, B.Cu at (327.6, 120.2)
- added U30: ESC, hot_swap_footprints:esc, B.Cu at (327.6, 160.2)
- added U31: ESC, hot_swap_footprints:esc, B.Cu at (264.6, 160.3)
- added U32: ESC, hot_swap_footprints:esc, B.Cu at (285.7, 160.2)
- added U33: ESC, hot_swap_footprints:esc, B.Cu at (306.6, 160.1)
- C12, C13, R30, R31: moved to F.Cu
- NT1: value Net-Tie_4 -> net-tie
- TP10, TP11, TP12, TP13, TP3, TP4, TP5, TP6, TP7, TP8, TP9: moved to B.Cu
- U23, U24, U25: footprint 5_Connectors_AMASS:AMASS_XT60-F_1x02_P7.20mm_Vertical -> 5_Connectors_AMASS:AMASS_XT30U-F_1x02_P5.0mm_Vertical
- moved R38 195.0 mm to (181.2, 148.1), turned to 90 degrees
- moved U7 192.1 mm to (211.9, 147.2), turned to 0 degrees
- moved U5 181.7 mm to (202.8, 158.4), turned to -90 degrees
- moved U6 181.1 mm to (212.7, 158.4), turned to -90 degrees
- moved C12 178.2 mm to (206.8, 159.8), turned to -90 degrees
- moved R30 178.1 mm to (207.3, 157.4)
- moved R35 177.8 mm to (202.3, 155.6), turned to 180 degrees
- moved U18 177.7 mm to (211.0, 174.2), turned to 90 degrees
- moved R31 177.6 mm to (217.2, 157.4)
- moved R34 177.6 mm to (205.2, 155.6), turned to 180 degrees
- moved C13 177.5 mm to (216.7, 159.8), turned to -90 degrees
- moved R37 177.0 mm to (212.3, 155.5), turned to 180 degrees
- moved R36 176.9 mm to (215.2, 155.5), turned to 180 degrees
- moved R39 175.1 mm to (182.7, 148.1), turned to 90 degrees
- moved D9 172.2 mm to (202.2, 115.8)
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Connections:
- D7 pad 1: GND -> GNDD
- R41 pad 1: +3V3 -> 3-3V_2
- R42 pad 1: +3V3 -> 3-3V_2
- R43 pad 1: +3V3 -> 3-3V_2
- R46 pad 1: +5V -> 5V_2
- R47 pad 1: +5V -> 5V_2
- TP12 pad 1: /batt_ctl/BATT_2_CTL -> /batt_ctl/BATT_2_VSENSE
- TP13 pad 1: GND -> GNDD
- TP8 pad 1: /batt_ctl/BATT_2_VSENSE -> /batt_ctl/BATT_2_CURR
- U15 pad 1: /batt_ctl/BATT_1_PWR -> GND
- U15 pad 2: GND -> /batt_ctl/BATT_1_PWR
- U16 pad 1: /batt_ctl/BATT_2_PWR -> GND
- U16 pad 2: GND -> /batt_ctl/BATT_2_PWR
- U17 pad 1: +3V3 -> GND
- U17 pad 2: GND -> +3V3
- U18 pad 1: 3-3V_2 -> GND
- U18 pad 2: GND -> 3-3V_2
- U19 pad 1: 3-3V_3 -> GND
- U19 pad 2: GND -> 3-3V_3
- U20 pad 1: +5V -> GND
- U20 pad 2: GND -> +5V
- U21 pad 1: 5V_2 -> GND
- U21 pad 2: GND -> 5V_2
- U22 pad 1: 5V_3 -> GND
- U22 pad 2: GND -> 5V_3
- U23 pad 1: +12V -> GND
- U23 pad 2: GND -> +12V
- U24 pad 1: 12V_2 -> GND
- U24 pad 2: GND -> 12V_2
- U25 pad 1: 12V_3 -> GND
- U25 pad 2: GND -> 12V_3
Other:
- board size 120 x 80 mm -> 190 x 80 mm

Commit message: updates
Parts:
- added C33: 1uF, 2_Passives_Capacitors_SMD_IPC:C_1608_603_B, F.Cu at (183.7, 152.5)
- added C34: 100pF, 2_Passives_Capacitors_SMD_IPC:C_1608_603_B, F.Cu at (175.9, 150.1)
- added C35: 1uF, 2_Passives_Capacitors_SMD_IPC:C_1608_603_B, F.Cu at (177.5, 147.2)
- added C36: 10uF, 2_Passives_Capacitors_SMD_IPC:C_1608_603_B, F.Cu at (179.0, 147.2)
- added C37: 10uF, 2_Passives_Capacitors_SMD_IPC:C_2012_805_B, F.Cu at (216.9, 145.1)
- added C38: 10uF, 2_Passives_Capacitors_SMD_IPC:C_1608_603_B, F.Cu at (233.3, 137.1)
- added D12: D_Schottky, 1_Semi_Discrete_Diodes_SMD:D_SOD-123F, F.Cu at (180.9, 146.4)
- added D13: LED, 1_Semi_Discrete_Diodes_SMD:D_0603, F.Cu at (232.5, 116.0)
- added D14: LED, 1_Semi_Discrete_Diodes_SMD:D_0603, F.Cu at (240.0, 164.4)
- added D15: LED, 1_Semi_Discrete_Diodes_SMD:D_0603, F.Cu at (241.4, 116.1)
- added D16: LED, 1_Semi_Discrete_Diodes_SMD:D_0603, F.Cu at (249.1, 164.4)
- added Q13: PMOS_SGD, 1_Semi_TO_SOT:VDFN-8, F.Cu at (198.7, 161.6)
- added Q14: PMOS_SGD, 1_Semi_TO_SOT:VDFN-8, F.Cu at (198.7, 165.8)
- added Q15: PMOS_SGD, 1_Semi_TO_SOT:VDFN-8, F.Cu at (197.7, 109.9)
- added Q16: PMOS_SGD, 1_Semi_TO_SOT:VDFN-8, F.Cu at (197.7, 105.7)
- added R62: 1k, 2_Passives_Resistors_SMD_IPC:R_1608_603_B, F.Cu at (197.7, 158.1)
- added R63: 1k, 2_Passives_Resistors_SMD_IPC:R_1608_603_B, F.Cu at (199.7, 169.2)
- added R64: 1k, 2_Passives_Resistors_SMD_IPC:R_1608_603_B, F.Cu at (198.7, 113.4)
- added R65: 1k, 2_Passives_Resistors_SMD_IPC:R_1608_603_B, F.Cu at (196.7, 102.2)
- added R66: 300, 2_Passives_Resistors_SMD_IPC:R_1608_603_B, F.Cu at (235.5, 117.4)
- added R67: 300, 2_Passives_Resistors_SMD_IPC:R_1608_603_B, F.Cu at (235.5, 116.0)
- added R68: 500, 2_Passives_Resistors_SMD_IPC:R_2012_805_B, F.Cu at (243.2, 164.4)
- added R69: 500, 2_Passives_Resistors_SMD_IPC:R_2012_805_B, F.Cu at (245.6, 116.2)
- added R70: 500, 2_Passives_Resistors_SMD_IPC:R_2012_805_B, F.Cu at (252.2, 164.4)
- added U34: AP2213-8_SOIC, 1_Semi_Misc:SOIC-8_3.9x4.9mm_P1.27mm, F.Cu at (180.2, 152.4)
- added U35: XT90PW-M, 5_Connectors_AMASS:AMASS_XT30U-F_1x02_P5.0mm_Vertical, F.Cu at (232.3, 106.2)
- added U36: LM1085-5.0, 1_Semi_TO_SOT:TO-263-3_TabPin2, F.Cu at (226.3, 143.6)
- C29, R48, U13: moved to F.Cu
- D1, D2: footprint 1_Semi_Discrete_Diodes_SMD:D_SOD-323 -> 1_Semi_Discrete_Diodes_SMD:D_SOD-123F
- D10, D11, D3, D4, D5, D6, D7, D8, D9: footprint 2_Passives_Resistors_SMD_IPC:R_1608_603_B -> 1_Semi_Discrete_Diodes_SMD:D_0603
- IC1: footprint 1_Semi_Misc:PSON50P200X300X50-9N -> 1_Semi_Misc:SOIC-8_3.9x4.9mm_P1.27mm
- SW1: footprint 3_Electromechanical_Buttons_Switches_SMD:CK_PTS645_SMD -> 3_Electromechanical_Buttons_Switches_SMD:KMR243GLFG
- moved R48 117.4 mm to (245.9, 132.2), turned to 180 degrees
- moved U13 112.9 mm to (244.4, 134.2), turned to 180 degrees
- moved C10 108.8 mm to (300.6, 150.7)
- moved C29 108.6 mm to (241.5, 134.1), turned to -90 degrees
- moved C5 108.0 mm to (300.4, 130.0)
- moved U25 68.1 mm to (249.0, 174.1), turned to 90 degrees
- moved R29 56.4 mm to (230.7, 154.4), turned to 180 degrees
- moved R32 55.2 mm to (228.6, 152.7), turned to 180 degrees
- moved C11 54.0 mm to (230.2, 156.7), turned to -90 degrees
- moved R33 51.9 mm to (225.7, 152.7), turned to 180 degrees
- moved U4 50.1 mm to (226.2, 155.5), turned to -90 degrees
- moved R39 47.5 mm to (228.2, 161.6), turned to -90 degrees
- moved C14 46.9 mm to (225.3, 158.4), turned to 0 degrees
- moved R38 45.3 mm to (224.7, 160.8), turned to 180 degrees
- moved D7 44.9 mm to (223.7, 162.4)
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Connections:
- net /batt_ctl/BATT_2_PWR renamed BATT_2_PWR
- C1 pad 1: /processor/VIN -> +3V3
- C1 pad 2: GND -> GNDD
- C11 pad 2: GNDD -> GND
- C14 pad 1: +3V3 -> 3-3V_1
- C14 pad 2: GNDD -> GND
- C29 pad 1: GNDD -> GND
- C29 pad 2: +3V3 -> 3-3V_1
- C31 pad 1: /processor/VIN -> +3V3
- C31 pad 2: GND -> GNDD
- C32 pad 1: /processor/VIN -> +3V3
- C32 pad 2: GND -> GNDD
- D1 pad 1: /processor/VIN -> Net-(C33-Pad2)
- D1 pad 2: +3V3 -> VUSB
- D2 pad 1: /processor/VIN -> Net-(C33-Pad2)
- D2 pad 2: VUSB -> BATT_1_PWR
- D7 pad 1: GNDD -> GND
- IC2 pad 10: /batt_ctl/BATT_2_VSENSE -> /batt_ctl/BATT_2_CURR
- IC2 pad 17: /processor/VIN -> +3V3
- IC2 pad 26: /batt_ctl/BATT_1_CTL -> /batt_ctl/BATT_2_CTL
- IC2 pad 27: /batt_ctl/BATT_2_CTL -> /batt_ctl/BATT_1_CTL
- IC2 pad 36: /processor/VIN -> +3V3
- IC2 pad 44: /processor/VIN -> +3V3
- IC2 pad 6: /processor/VIN -> +3V3
- IC2 pad 9: /batt_ctl/BATT_2_CURR -> /batt_ctl/BATT_2_VSENSE
- J1 pad 1: /RESET -> /~{RESET_RAW}
- J7 pad 6: GND -> GNDD
- P2 pad 1: /RESET -> /~{RESET_RAW}
- R17 pad 1: /batt_ctl/BATT_1_PWR -> BATT_1_PWR
- R32 pad 1: +3V3 -> 3-3V_1
- R33 pad 2: GNDD -> GND
- R38 pad 1: +3V3 -> 3-3V_1
- R39 pad 1: +3V3 -> 3-3V_1
- R40 pad 1: +3V3 -> 3-3V_1
- R48 pad 2: +3V3 -> 3-3V_1
- R5 pad 1: /batt_ctl/BATT_1_PWR -> BATT_1_PWR
- U1 pad 10: /RESET -> /~{RESET_RAW}
- U13 pad 4: GNDD -> GND
- U13 pad 8: +3V3 -> 3-3V_1
- U13 pad 9: GNDD -> GND
- U15 pad 2: /batt_ctl/BATT_1_PWR -> BATT_1_PWR
- U17 pad 2: +3V3 -> 3-3V_1
- U2 pad 6: /batt_ctl/BATT_1_PWR -> BATT_1_PWR
- U4 pad 14: GNDD -> GND
- U4 pad 3: GNDD -> GND
- U4 pad 9: +3V3 -> 3-3V_1
Routing:
- net GND: track 0.00 -> 214.1 mm, vias 0 -> 51
- net /SCL: track 0.00 -> 164.6 mm, vias 0 -> 3
- net /SDA: track 0.00 -> 164.6 mm, vias 0 -> 3
- net +BATT: track 0.00 -> 127.1 mm, vias 0 -> 34
- net GNDD: track 0.00 -> 118.1 mm, vias 1 -> 26
- net +5V: track 0.00 -> 88.3 mm, vias 0 -> 3
- net /batt_ctl/BATT_1_CTL: track 0.00 -> 73.8 mm, vias 0 -> 2
- net BATT_2_PWR: track 0.00 -> 65.8 mm, vias 0 -> 4
- net 3-3V_1: track 0.00 -> 63.6 mm, vias 0 -> 2
- net /~{RESET_RAW}: track 0.00 -> 59.0 mm, vias 0 -> 2
- net /batt_ctl/BATT_2_CTL: track 0.00 -> 50.5 mm, vias 0 -> 2
- net 5V_2: track 0.00 -> 42.5 mm
- net +3V3: track 0.00 -> 41.8 mm, vias 1 -> 17
- net Net-(Q2-Pad3): track 0.00 -> 41.4 mm
- net /batt_ctl/BATT_1_CURR: track 0.00 -> 40.4 mm, vias 0 -> 2
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Other:
- board size 190 x 80 mm -> 200 x 80 mm
- board text added: "12V - 3A"
- board text added: "3V"
- board text added: "3V - 1.2A"
- board text added: "5V"
- board text added: "5V - 3A"
