File: 1.0/1.0.kicad_sch (KiCad schematic)
At the start: 9 parts

Commit message: updates
Parts:
- removed J?: header_01x04, symbol 5.connector.interconnect:header_01x04
- removed J? (x2): header_01x02, symbol 5.connector.interconnect:header_01x02
- removed J?: header_01x05, symbol 5.connector.interconnect:header_01x05
- removed NT?: net-tie, symbol 0.power-symbols:net-tie
- added J1: header_01x04, 5_Connectors_misc:Stemma_QT_V, symbol 5.connector.interconnect:header_01x04
- added J3, J4, J5, J6: header_01x04, 5_Connectors_misc:Stemma_QT_2, symbol 5.connector.interconnect:header_01x04
- added JP1, JP2: Jumper_NO_Dual, 0_misc:SolderJumper-3_P1.3mm_Open_RoundedPad1.0x1.5mm_NumberLabels, symbol 2.passive:Jumper_NO_Dual
- added NT1: Net-Tie_4, 0_NetTie:NetTie-4_SMD_Pad2.0mm, symbol 2.passive:Net-Tie_4
- added U15, U16: XT90PW-M, 5_Connectors_AMASS:AMASS_XT90PW-M_Horizontal, symbol 5.connector.interconnect:XT90PW-M
- added U17, U18, U19, U20, U21, U22: XT90PW-M, 5_Connectors_AMASS:AMASS_XT30U-F_1x02_P5.0mm_Vertical, symbol 5.connector.interconnect:XT90PW-M
- added U23, U24, U25: XT90PW-M, 5_Connectors_AMASS:AMASS_XT60-F_1x02_P7.20mm_Vertical, symbol 5.connector.interconnect:XT90PW-M
- J2: renamed from J?; footprint (none) -> 5_Connectors_misc:amphenol_micro_usb_no_flange_10118192
- gave numbers to parts that had none: 3
Connections:
- net +3V3: now also J5.2, J6.2, JP1.1, JP2.1, U17.1 (+)
- net GND: now also NT1.2, NT1.4, U15.2 (-), U16.2 (-), U17.2 (-), U18.2 (-), U19.2 (-), U20.2 (-), U21.2 (-), U22.2 (-), U23.2 (-), U24.2 (-), U25.2 (-)
- net GNDD: now also J1.4, J3.2, J4.2, J5.1, J6.1, NT1.1, NT1.3
- net RESET: now also J1.1
- net SCL: now also J5.4, J6.4
- net SDA: now also J5.3, J6.3
- net SERIAL1_RX: now also J1.3
- net SERIAL1_TX: now also J1.2
- net USB_D+: now also J2.3 (D+)
- net USB_D-: now also J2.2 (D-)
- net batt_ctl/BATT_1_PWR: now also U15.1 (+)
- net batt_ctl/BATT_2_PWR: now also U16.1 (+)
- new net: J4.1, JP2.2
- new net: J3.1, JP1.2
- new net +12V: U23.1 (+)
- new net +5V: JP1.3, JP2.3, U20.1 (+)
- new net 12V_2: U24.1 (+)
- new net 12V_3: U25.1 (+)
- new net 3-3V_2: U18.1 (+)
- new net 3-3V_3: U19.1 (+)
- new net 5V_2: U21.1 (+)
- new net 5V_3: U22.1 (+)
- new net A0_SENSE: J3.3
- new net A5_SENSE: J4.3
- no-connect marks 2 -> 4
Other:
- sheet processor ports: added A0_SENSE, A5_SENSE, ~{RESET_RAW}; removed none
- note added: "12V @ 3A"
- note added: "3.3V @ 1.2A"
- note added: "5V @ 3A"
- note added: "Analog Inputs"
- note added: "Route outputs parallel with thermal vias"
- moved on the sheet: J2, P1, P2, U1

Commit message: updates
Parts:
- NT1: footprint 0_NetTie:NetTie-4_SMD_Pad2.0mm -> 0_NetTie:NetTie-2_SMD_Pad2.0mm
Other:
- moved on the sheet: J1, J2, J3, J4, J5, J6, JP1, JP2, NT1, P1, P2, U1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

Commit message: updates
Parts:
- removed NT1: Net-Tie_4, 0_NetTie:NetTie-2_SMD_Pad2.0mm, symbol 2.passive:Net-Tie_4
- added J10, J11, J12, J13, J14, J15, J8, J9: header_01x03, 5_Connectors_Molex:MegaF_RAH_Single_3x5.7mm, symbol 5.connector.interconnect:header_01x03
- added NT1: net-tie, 0_NetTie:NetTie-2_SMD_Pad2.0mm, symbol 0.power-symbols:net-tie
- added U26, U27, U28, U29, U30, U31, U32, U33: ESC, hot_swap_footprints:esc, symbol symbols:ESC
- U23, U24, U25: footprint 5_Connectors_AMASS:AMASS_XT60-F_1x02_P7.20mm_Vertical -> 5_Connectors_AMASS:AMASS_XT30U-F_1x02_P5.0mm_Vertical
Connections:
- net +12V: now also U23.2 (+); no longer U23.1 (+)
- net +3V3: now also U17.2 (+); no longer U17.1 (+)
- net +5V: now also U20.2 (+); no longer U20.1 (+)
- net +BATT: now also U26.1 (PWR), U27.1 (PWR), U28.1 (PWR), U29.1 (PWR), U30.1 (PWR), U31.1 (PWR), U32.1 (PWR), U33.1 (PWR)
- net 12V_2: now also U24.2 (+); no longer U24.1 (+)
- net 12V_3: now also U25.2 (+); no longer U25.1 (+)
- net 3-3V_2: now also U18.2 (+); no longer U18.1 (+)
- net 3-3V_3: now also U19.2 (+); no longer U19.1 (+)
- net 5V_2: now also U21.2 (+); no longer U21.1 (+)
- net 5V_3: now also U22.2 (+); no longer U22.1 (+)
- net GND: now also U15.1 (-), U16.1 (-), U17.1 (-), U18.1 (-), U19.1 (-), U20.1 (-), U21.1 (-), U22.1 (-), U23.1 (-), U24.1 (-), U25.1 (-), NT1.2, U26.2 (GND), U27.2 (GND), U28.2 (GND), U29.2 (GND), U30.2 (GND), U31.2 (GND), U32.2 (GND), U33.2 (GND); no longer U15.2 (-), U16.2 (-), U17.2 (-), U18.2 (-), U19.2 (-), U20.2 (-), U21.2 (-), U22.2 (-), U23.2 (-), U24.2 (-), U25.2 (-)
- net GNDD: now also NT1.1
- net batt_ctl/BATT_1_PWR: now also U15.2 (+); no longer U15.1 (+)
- net batt_ctl/BATT_2_PWR: now also U16.2 (+); no longer U16.1 (+)
- new net: J9.1, U27.5 (P1)
- new net: J9.2, U27.4 (P2)
- new net: J9.3, U27.3 (P3)
- new net: J10.3, U28.3 (P3)
- new net: J10.2, U28.4 (P2)
- new net: J10.1, U28.5 (P1)
- new net: J8.3, U26.3 (P3)
- new net: J8.2, U26.4 (P2)
- new net: J8.1, U26.5 (P1)
- new net: J12.1, U30.5 (P1)
- new net: J12.2, U30.4 (P2)
- new net: J12.3, U30.3 (P3)
- new net: J13.3, U31.3 (P3)
- new net: J13.2, U31.4 (P2)
- new net: J13.1, U31.5 (P1)
- new net: J14.3, U32.3 (P3)
- new net: J14.2, U32.4 (P2)
- new net: J14.1, U32.5 (P1)
- new net: J15.3, U33.3 (P3)
- new net: J15.2, U33.4 (P2)
- new net: J15.1, U33.5 (P1)
- new net: J11.1, U29.5 (P1)
- new net: J11.2, U29.4 (P2)
- new net: J11.3, U29.3 (P3)
Other:
- note added: "ESC Interface"

Commit message: updates
Parts:
- added U35: XT90PW-M, 5_Connectors_AMASS:AMASS_XT30U-F_1x02_P5.0mm_Vertical, symbol 5.connector.interconnect:XT90PW-M
Connections:
- net +3V3: no longer U17.2 (+)
- net GND: now also U35.1 (-)
- net RESET: no longer J1.1, P2.1, U1.10 (~{RESET})
- net ~{RESET_RAW}: now also J1.1, P2.1, U1.10 (~{RESET})
- net batt_ctl/BATT_1_PWR renamed BATT_1_PWR
- net batt_ctl/BATT_2_PWR renamed BATT_2_PWR
- new net 3-3V_1: U17.2 (+)
- new net 5V_4: U35.2 (+)
Other:
- moved on the sheet: U15, U16, U17, U18, U19, U20, U21, U22, U23, U24, U25
