File: 1.0/batt_ctl.kicad_sch (KiCad schematic)
At the start: 40 parts

Commit message: updates
Parts:
- removed C?: 1uF, symbol 2.passive:C
- removed C? (x2): 470uF, 0_misc:THT_470uF_Cap, symbol 2.passive:CP1
- removed C?: 0.1uF, symbol 2.passive:C
- removed D?: LED, symbol 1.semi.opto:LED
- removed Q? (x4): PMOS_SGD, 1_Semi_TO_SOT:VDFN-8, symbol 1.semi.discrete:Q_NMOS_SGD
- removed Q? (x2): BC847, 1.Semi.TO_SOT:SOT-23, symbol 1.semi.discrete:BC847
- removed R? (x7): 1k, symbol 2.passive:R
- removed R?: 470, symbol 2.passive:R
- removed R?: 10k, symbol 2.passive:R
- removed R? (x3): 4k7, symbol 2.passive:R
- removed U?: ACS781, 1_Semi_TO_SOT:7-LR-PSOF, symbol 1.semi.ic.sensor:ACS781
- added C10, C5, C6, C9: 470uF, 0_misc:THT_470uF_Cap, symbol 2.passive:CP
- added C7: 0.1uF, 2_Passives_Capacitors_SMD_IPC:C_1608_603_B, symbol 2.passive:C
- added C8: 1uF, 2_Passives_Capacitors_SMD_IPC:C_1608_603_B, symbol 2.passive:C
- added Q10, Q11, Q12, Q3, Q4, Q5, Q6, Q9: PMOS_SGD, 1_Semi_TO_SOT:VDFN-8, symbol 1.semi.discrete:Q_NMOS_SGD
- added Q2, Q7: BC847, 1_Semi_TO_SOT:SOT-23, symbol 1.semi.discrete:BC847
- added R11, R25, R27, R8: 500, 2_Passives_Resistors_SMD_IPC:R_2012_805_B, symbol 2.passive:R
- added R12, R13, R14, R21, R22, R28, R54, R55, R56, R57: 1k, 2_Passives_Resistors_SMD_IPC:R_1608_603_B, symbol 2.passive:R
- added R23: 10k, 2_Passives_Resistors_SMD_IPC:R_1608_603_B, symbol 2.passive:R
- added R24, R26: 4k7, 2_Passives_Resistors_SMD_IPC:R_1608_603_B, symbol 2.passive:R
- added U3: ACS781, 1_Semi_TO_SOT:7-LR-PSOF, symbol 1.semi.ic.sensor:ACS781
- C3, C4: renamed from C?; footprint (none) -> 2_Passives_Capacitors_SMD_IPC:C_1608_603_B
- D3, D4, D5: renamed from D?; footprint (none) -> 2_Passives_Resistors_SMD_IPC:R_1608_603_B
- R10: renamed from R?; value 1k -> 4k7; footprint (none) -> 2_Passives_Resistors_SMD_IPC:R_1608_603_B
- R15, R17, R18, R19, R20, R5, R6, R7, R9: renamed from R?; footprint (none) -> 2_Passives_Resistors_SMD_IPC:R_1608_603_B
- gave numbers to parts that had none: 1
Connections:
- net +3V3: now also C7.2, U3.1 (VCC)
- net BATT_1_CTL: now also R8.1; no longer R10.2
- net BATT_1_PWR: now also R17.1
- net BATT_2_CTL: now also R23.2, R25.1
- net BATT_2_CURR: now also R24.1
- net BATT_2_PWR: now also R19.1, U3.6 (IP-)
- net GND: now also C10.2, C5.2, C6.2, C9.2
- net GNDD: now also C7.1, C8.1, Q2.2 (E), Q7.2 (E), R23.1, U3.2 (GND)
- net at U2.5 (IP+): now also Q3.3 (D), Q4.3 (D), Q5.3 (D), Q6.3 (D), R11.2
- net at R10.1: now also Q2.1 (B)
- net +15V renamed +BATT
- net +BATT: now also C10.1, C5.1, C6.1, C9.1, Q10.1 (S), Q11.1 (S), Q12.1 (S), Q3.1 (S), Q4.1 (S), Q5.1 (S), Q6.1 (S), Q9.1 (S)
- new net: Q7.1 (B), R26.1
- new net: Q7.3 (C), R28.1, R54.2, R55.2, R56.2, R57.2
- new net: C8.2, R24.2, U3.3 (VOUT)
- new net: Q10.2 (G), R55.1
- new net: Q10.3 (D), Q11.3 (D), Q12.3 (D), Q9.3 (D), R27.2, U3.5 (IP+)
- new net: R25.2, R26.2
- new net: Q6.2 (G), R22.1
- new net: Q2.3 (C), R12.1, R13.2, R14.2, R21.2, R22.2
- new net: Q11.2 (G), R56.1
- new net: Q12.2 (G), R57.1
- new net: Q3.2 (G), R13.1
- new net: R10.2, R8.2
- new net: Q5.2 (G), R21.1
- new net: Q9.2 (G), R54.1
- new net: R27.1, R28.2
- new net: Q4.2 (G), R14.1
- new net: R11.1, R12.2
Other:
- note added: "Green"
- note removed: "Blue"
- moved on the sheet: C3, C4, D5, R10, R15, R17, R18, R19, R20, R6, R7, U2

Commit message: updates
Parts:
- added Q13, Q14, Q15, Q16: PMOS_SGD, 1_Semi_TO_SOT:VDFN-8, symbol 1.semi.discrete:Q_NMOS_SGD
- added R62, R63, R64, R65: 1k, 2_Passives_Resistors_SMD_IPC:R_1608_603_B, symbol 2.passive:R
- D3, D4, D5: footprint 2_Passives_Resistors_SMD_IPC:R_1608_603_B -> 1_Semi_Discrete_Diodes_SMD:D_0603
Connections:
- net +BATT: now also Q13.1 (S), Q14.1 (S), Q15.1 (S), Q16.1 (S)
- net at Q7.3 (C), R28.1, R54.2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: now also R64.2, R65.2
- net at Q10.3 (D), Q11.3 (D), Q12.3 (D)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: now also Q15.3 (D), Q16.3 (D)
- net at Q2.3 (C), R12.1, R13.2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: now also R62.2, R63.2
- net at Q3.3 (D), Q4.3 (D), Q5.3 (D)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: now also Q13.3 (D), Q14.3 (D)
- new net: Q15.2 (G), R64.1
- new net: Q16.2 (G), R65.1
- new net: Q14.2 (G), R63.1
- new net: Q13.2 (G), R62.1
Other:
- moved on the sheet: C10, C3, C4, C5, C6, C7, C8, C9, D3, D4, D5, Q10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
