File: 1.0/peripherals.kicad_sch (KiCad schematic)
At the start: 10 parts

Commit message: updates
Parts:
- removed Q?: BC847, 1.Semi.TO_SOT:SOT-23, symbol 1.semi.discrete:BC847
- removed R?: 300, symbol 2.passive:R
- removed R?: 10k, symbol 2.passive:R
- removed SP?: buzzer, symbol 3.electromechanical.audio:buzzer
- removed U? (x2): BME280, Package_LGA:Bosch_LGA-8_2.5x2.5mm_P0.65mm_ClockwisePinNumbering, symbol 1.semi.ic.sensor:BME280
- added C29, C30: 0.1uF, 2_Passives_Capacitors_SMD_IPC:C_1608_603_B, symbol 2.passive:C
- added Q8: BC847, 1_Semi_TO_SOT:SOT-23, symbol 1.semi.discrete:BC847
- added R48, R53: 10k, 2_Passives_Resistors_SMD_IPC:R_1608_603_B, symbol 2.passive:R
- added R51, R52: 500, 2_Passives_Resistors_SMD_IPC:R_2012_805_B, symbol 2.passive:R
- added U13, U14: PCT2075, 1_Semi_Misc:PCT2075TP_147, symbol 1.semi.ic.sensor:PCT2075
- R49, R50: renamed from R?; footprint (none) -> 2_Passives_Resistors_SMD_IPC:R_1608_603_B
- SP1: renamed from SP?; footprint (none) -> 3_Electromechanical_Audio:13-9mm_Buzzer
- gave numbers to parts that had none: 1
Connections:
- net +3V3: now also C29.2, C30.2, R48.2, R53.2, U13.8 (VCC), U14.8 (VCC)
- net BUZZER: now also R49.2
- net GNDD: now also C29.1, C30.1, Q8.2 (E), U13.4 (GND), U13.9 (EP_GND), U14.4 (GND), U14.5 (A2), U14.6 (A1), U14.7 (A0), U14.9 (EP_GND)
- net SCL: now also U13.2 (SCL), U14.2 (SCL)
- net SDA: now also U13.1 (SDA), U14.1 (SDA)
- net at R50.1: now also Q8.1 (B); no longer R49.2
- net at SP1.1 (+): now also Q8.3 (C), R51.2, R52.2
- new net: R48.1, U13.3 (OS)
- new net: R53.1, U14.3 (OS)
- new net +5V: R51.1, R52.1
- no-connect marks 4 -> 5
Other:
- note added: "I2C: 0x37"
- note added: "I2C: 0x48"
- note removed: "0x76"
- note removed: "0x77"
- moved on the sheet: R49, R50, SP1

Commit message: updates
Connections:
- net +3V3: no longer C29.2, R48.2, U13.8 (VCC)
- net GND: now also C29.1, U13.4 (GND), U13.9 (EP_GND); no longer J7.6 (GND)
- net GNDD: now also J7.6 (GND); no longer C29.1, U13.4 (GND), U13.9 (EP_GND)
- new net 3-3V_1: C29.2, R48.2, U13.8 (VCC)
Changed lines of the file:
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@@
   (junction (at 55.245 53.34) (diameter 0) (color 0 0 0 0)
-  )
-  (junction (at 102.235 129.54) (diameter 0) (color 0 0 0 0)
   )
   (junction (at 185.42 91.44) (diameter 0) (color 0 0 0 0)
@@
     (stroke (width 0) (type default) (color 0 0 0 0))
   )
-  (wire (pts (xy 102.235 129.54) (xy 110.49 129.54))
-    (stroke (width 0) (type default) (color 0 0 0 0))
-  )
   (wire (pts (xy 89.535 66.04) (xy 88.265 66.04))
     (stroke (width 0) (type default) (color 0 0 0 0))
@@
   )
   (wire (pts (xy 42.545 76.2) (xy 42.545 77.47))
+    (stroke (width 0) (type default) (color 0 0 0 0))
+  )
+  (wire (pts (xy 38.1 53.34) (xy 41.275 53.34))
     (stroke (width 0) (type default) (color 0 0 0 0))
   )
@@
   (text "Thermometers" (at 65.405 41.275 0)
     (effects (font (size 3 3)) (justify left bottom))
+  )
+  (global_label "3-3V_1" (shape input) (at 41.275 52.07 90) (fields_autoplaced)
+    (effects (font (size 1.27 1.27)) (justify left))
+    (property "Intersheet References" "${INTERSHEET_REFS}" (id 0) (at 41.1956 42.3998 90)
+      (effects (font (size 1.27 1.27)) (justify left) hide)
+    )
   )
   (hierarchical_label "MOSI" (shape input) (at 103.505 121.92 0)
@@
     (pin "9")
   )
-  (symbol (lib_id "0.power-symbols:+3.3V") (at 41.275 52.07 0) (unit 1)
-    (in_bom yes) (on_board yes) (fields_autoplaced)
-    (property "Reference" "#PWR061" (id 0) (at 41.275 55.88 0)
-      (effects (font (size 1.27 1.27)) hide)
-    )
-    (property "Value" "+3.3V" (id 1) (at 41.275 48.4655 0))
-    (property "Footprint" "" (id 2) (at 41.275 52.07 0)
-      (effects (font (size 1.27 1.27)) hide)
-    )
-    (property "Datasheet" "" (id 3) (at 41.275 52.07 0)
-      (effects (font (size 1.27 1.27)) hide)
-    )
-    (pin "1")
-  )
   (symbol (lib_id "2.passive:R") (at 172.72 82.55 270) (unit 1)
     (in_bom yes) (on_board yes) (fields_autoplaced)
@@
     (pin "1")
     (pin "2")
-  )
-  (symbol (lib_id "0.power-symbols:PWR_FLAG") (at 110.49 129.54 270) (unit 1)
-    (in_bom yes) (on_board yes) (fields_autoplaced)
-    (property "Reference" "#FLG06" (id 0) (at 112.395 129.54 0)
-      (effects (font (size 1.27 1.27)) hide)
-    )
-    (property "Value" "PWR_FLAG" (id 1) (at 113.665 129.9738 90)
-      (effects (font (size 1.27 1.27)) (justify left))
-    )
-    (property "Footprint" "" (id 2) (at 110.49 129.54 0)
-      (effects (font (size 1.27 1.27)) hide)
-    )
-    (property "Datasheet" "" (id 3) (at 110.49 129.54 0)
-      (effects (font (size 1.27 1.27)) hide)
-    )
-    (pin "1")
   )
   (symbol (lib_id "1.semi.ic.sensor:PCT2075") (at 41.275 58.42 0) (unit 1)
@@
     (pin "2")
   )
-  (symbol (lib_id "0.power-symbols:GNDD") (at 40.005 78.74 0) (unit 1)
-    (in_bom yes) (on_board yes) (fields_autoplaced)
-    (property "Reference" "#PWR04" (id 0) (at 40.005 85.09 0)
-      (effects (font (size 1.27 1.27)) hide)
-    )
-    (property "Value" "GNDD" (id 1) (at 40.005 83.1834 0))
+  (symbol (lib_id "2.passive:R") (at 55.245 60.325 180) (unit 1)
+    (in_bom yes) (on_board yes) (fields_autoplaced)
+    (property "Reference" "R48" (id 0) (at 57.023 59.4903 0)
+      (effects (font (size 1.27 1.27)) (justify right))
+    )
+    (property "Value" "10k" (id 1) (at 57.023 62.0272 0)
+      (effects (font (size 1.27 1.27)) (justify right))
+    )
+    (property "Footprint" "2_Passives_Resistors_SMD_IPC:R_1608_603_B" (id 2) (at 57.023 60.325 90)
+      (effects (font (size 1.27 1.27)) hide)
+    )
+    (property "Datasheet" "~" (id 3) (at 55.245 60.325 0)
+      (effects (font (size 1.27 1.27)) hide)
+    )
+    (pin "1")
+    (pin "2")
+  )
+  (symbol (lib_id "0.power-symbols:GND") (at 40.005 78.74 0) (unit 1)
+    (in_bom yes) (on_board yes) (fields_autoplaced)
+    (property "Reference" "#PWR0157" (id 0) (at 40.005 85.09 0)
+      (effects (font (size 1.27 1.27)) hide)
+    )
+    (property "Value" "GND" (id 1) (at 40.005 83.1834 0))
     (property "Footprint" "" (id 2) (at 40.005 78.74 0)
       (effects (font (size 1.27 1.27)) hide)
@@
     )
     (pin "1")
-  )
-  (symbol (lib_id "2.passive:R") (at 55.245 60.325 180) (unit 1)
-    (in_bom yes) (on_board yes) (fields_autoplaced)
-    (property "Reference" "R48" (id 0) (at 57.023 59.4903 0)
-      (effects (font (size 1.27 1.27)) (justify right))
-    )
-    (property "Value" "10k" (id 1) (at 57.023 62.0272 0)
-      (effects (font (size 1.27 1.27)) (justify right))
-    )
-    (property "Footprint" "2_Passives_Resistors_SMD_IPC:R_1608_603_B" (id 2) (at 57.023 60.325 90)
-      (effects (font (size 1.27 1.27)) hide)
-    )
-    (property "Datasheet" "~" (id 3) (at 55.245 60.325 0)
-      (effects (font (size 1.27 1.27)) hide)
-    )
-    (pin "1")
-    (pin "2")
   )
   (symbol (lib_id "2.passive:R") (at 167.64 86.995 180) (unit 1)
@@
     (pin "3")
   )
+  (symbol (lib_id "0.power-symbols:GNDD") (at 102.235 130.81 0) (unit 1)
+    (in_bom yes) (on_board yes) (fields_autoplaced)
+    (property "Reference" "#PWR0122" (id 0) (at 102.235 137.16 0)
+      (effects (font (size 1.27 1.27)) hide)
+    )
+    (property "Value" "GNDD" (id 1) (at 102.235 135.2534 0))
+    (property "Footprint" "" (id 2) (at 102.235 130.81 0)
+      (effects (font (size 1.27 1.27)) hide)
+    )
+    (property "Datasheet" "" (id 3) (at 102.235 130.81 0)
+      (effects (font (size 1.27 1.27)) hide)
+    )
+    (pin "1")
+  )
   (symbol (lib_id "0.power-symbols:+5V") (at 185.42 65.405 0) (unit 1)
     (in_bom yes) (on_board yes) (fields_autoplaced)
@@
     (pin "1")
   )
-  (symbol (lib_id "0.power-symbols:GND") (at 102.235 130.81 0) (unit 1)
-    (in_bom yes) (on_board yes) (fields_autoplaced)
-    (property "Reference" "#PWR0122" (id 0) (at 102.235 137.16 0)
-      (effects (font (size 1.27 1.27)) hide)
-    )
-    (property "Value" "GND" (id 1) (at 102.235 135.2534 0))
-    (property "Footprint" "" (id 2) (at 102.235 130.81 0)
-      (effects (font (size 1.27 1.27)) hide)
-    )
-    (property "Datasheet" "" (id 3) (at 102.235 130.81 0)
-      (effects (font (size 1.27 1.27)) hide)
-    )
+  (symbol (lib_id "0.power-symbols:PWR_FLAG") (at 38.1 53.34 90) (unit 1)
+    (in_bom yes) (on_board yes) (fields_autoplaced)
+    (property "Reference" "#FLG0104" (id 0) (at 36.195 53.34 0)
+      (effects (font (size 1.27 1.27)) hide)
+    )
+    (property "Value" "PWR_FLAG" (id 1) (at 34.9251 53.7738 90)
+      (effects (font (size 1.27 1.27)) (justify left))
+    )
+    (property "Footprint" "" (id 2) (at 38.1 53.34 0)
+      (effects (font (size 1.27 1.27)) hide)
+    )
+    (property "Datasheet" "" (id 3) (at 38.1 53.34 0)
+      (effects (font (size 1.27 1.27)) hide)
+    )
