File: 1.0/power_reg.kicad_sch (KiCad schematic)
At the start: 38 parts

Commit message: updates
Parts:
- removed C? (x6): 10uF, 2_Passives_Capacitors_SMD_IPC:C_1608_603_B, symbol 2.passive:C
- removed C? (x2): 470uF, 0_misc:THT_470uF_Cap, symbol 2.passive:CP1
- removed D? (x3): LED, symbol 1.semi.opto:LED
- removed R? (x2): 22k, symbol 2.passive:R
- removed R? (x2): 115k, symbol 2.passive:R
- removed R? (x2): 470, symbol 2.passive:R
- removed R? (x2): 75k, symbol 2.passive:R
- removed R?: 300, symbol 2.passive:R
- removed U? (x2): LM1085, symbol 1.semi.ic.pmic.voltagereg:LM1085
- removed U? (x3): MPM3610, symbol 1.semi.ic.pmic.voltagereg:MPM3610
- added C12, C13, C17, C18, C19, C23, C24, C25: 10uF, 2_Passives_Capacitors_SMD_IPC:C_2012_805_B, symbol 2.passive:C
- added C16, C20, C22, C26, C27, C28: 10uF, 2_Passives_Capacitors_SMD_IPC:C_1608_603_B, symbol 2.passive:C
- added D10, D8, D9: LED, 2_Passives_Resistors_SMD_IPC:R_1608_603_B, symbol 1.semi.opto:LED
- added R31: 75k, 2_Passives_Resistors_SMD_IPC:R_1608_603_B, symbol 2.passive:R
- added R36: 102k, 2_Passives_Resistors_SMD_IPC:R_1608_603_B, symbol 2.passive:R
- added R37: 32.4k, 2_Passives_Resistors_SMD_IPC:R_1608_603_B, symbol 2.passive:R
- added R38, R39, R41, R42, R43, R44, R45, R46, R47: 300, 2_Passives_Resistors_SMD_IPC:R_1608_603_B, symbol 2.passive:R
- added U10, U11, U12: LM1085-3.0, 1_Semi_TO_SOT:TO-263-3_TabPin2, symbol 1.semi.ic.pmic.voltagereg:LM1085
- added U5, U6: MPM3610, 1_Semi_QFN:20-PowerLQFN, symbol 1.semi.ic.pmic.voltagereg:MPM3610
- added U7, U8, U9: LM1085-5.0, 1_Semi_TO_SOT:TO-263-3_TabPin2, symbol 1.semi.ic.pmic.voltagereg:LM1085
- C11: renamed from C?; footprint 2_Passives_Capacitors_SMD_IPC:C_1608_603_B -> 2_Passives_Capacitors_SMD_IPC:C_2012_805_B
- D7: renamed from D?; footprint (none) -> 2_Passives_Resistors_SMD_IPC:R_1608_603_B
- R29, R30, R32, R33, R34, R35, R40: renamed from R?; footprint (none) -> 2_Passives_Resistors_SMD_IPC:R_1608_603_B
- U4: renamed from U?; footprint (none) -> 1_Semi_QFN:20-PowerLQFN
- gave numbers to parts that had none: 3
Connections:
- net +12V: now also C28.1, U10.2 (VOUT)
- net +3V3: now also R38.1, R39.1, R41.1, R42.1, R43.1; no longer C15.1, R34.1, U4.7 (OUT), U4.8 (OUT)
- net +5V: now also R44.1, R45.1, R46.1, R47.1, U8.2 (VOUT)
- net GND: now also C12.2, C13.2, C16.2, C17.2, C18.2, C19.2, C20.2, C22.2, C23.2, C24.2, C25.2, C26.2, C27.2, C28.2, D10.1 (K), D8.1 (K), D9.1 (K), R37.2, U10.1 (ADJ), U11.1 (ADJ), U12.1 (ADJ), U7.1 (ADJ), U8.1 (ADJ), U9.1 (ADJ)
- net GNDD: now also U5.14 (PGND), U5.3 (AGND), U6.14 (PGND), U6.3 (AGND); no longer U4.12 (PGND), U4.13 (PGND)
- net at D7.2 (A), R40.2: now also R38.2, R39.2
- net at R34.2, R35.1: now also U5.1 (FB)
- net at R30.2: now also U5.17 (EN)
- net +15V renamed +BATT
- net +BATT: now also C12.1, C13.1, C17.1, C18.1, C19.1, C23.1, C24.1, C25.1, R31.1, U10.3 (VIN), U11.3 (VIN), U12.3 (VIN), U5.16 (IN), U6.16 (IN), U7.3 (VIN), U8.3 (VIN), U9.3 (VIN)
- new net: D8.2 (A), R41.2, R42.2, R43.2
- new net: D9.2 (A), R44.2, R45.2
- new net: D10.2 (A), R46.2, R47.2
- new net: R31.2, U6.17 (EN)
- new net: R36.2, R37.1, U6.1 (FB)
- new net 12V_2: C27.1, U11.2 (VOUT)
- new net 12V_3: C26.1, U12.2 (VOUT)
- new net 3-3V_2: C15.1, R34.1, U5.9 (OUT)
- new net 3-3V_3: C16.1, R36.1, U6.9 (OUT)
- new net 5V_2: C22.1, U9.2 (VOUT)
- new net 5V_3: C20.1, U7.2 (VOUT)
- no-connect marks 24 -> 30
Other:
- note added: "12V @ 3A"
- note added: "3.3V @ 1.2A"
- note added: "5V @ 3A"
- note added: "Add 16V 3A"
- note added: "Leave NC pins floating Refer to DS p18 for thermal considerations"
- note added: "Leave NC pins floating Refer to DS p21 for thermal considerations"
- note added: "add 24v 3a"
- note added: "add 48v 3a"
- note removed: "12V"
- note removed: "3.3V"
- note removed: "5V"
- note removed: "Leave NC pins floating"
- moved on the sheet: C14, C15, C21, D7, R40

Commit message: updates
Connections:
- net GND: now also U5.14 (PGND), U5.3 (AGND), U6.14 (PGND), U6.3 (AGND)
- net GNDD: no longer U5.14 (PGND), U5.3 (AGND), U6.14 (PGND), U6.3 (AGND)
Other:
- note added: "Digital Ground Regulator"
Changed lines of the file:
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@@
     (effects (font (size 1.27 1.27)) (justify left bottom))
+  )
+  (text "Digital Ground \nRegulator\n" (at 28.575 69.85 180)
+    (effects (font (size 1.27 1.27)) (justify right bottom))
   )
   (text "Leave NC pins floating\nRefer to DS p21 for \nthermal considerations"
@@
     )
     (property "Datasheet" "" (id 3) (at 250.19 52.07 0)
+      (effects (font (size 1.27 1.27)) hide)
+    )
+    (pin "1")
+  )
+  (symbol (lib_id "0.power-symbols:GND") (at 39.37 120.65 0) (unit 1)
+    (in_bom yes) (on_board yes)
+    (property "Reference" "#PWR031" (id 0) (at 39.37 127 0)
+      (effects (font (size 1.27 1.27)) hide)
+    )
+    (property "Value" "GND" (id 1) (at 39.37 125.0934 0))
+    (property "Footprint" "" (id 2) (at 39.37 120.65 0)
+      (effects (font (size 1.27 1.27)) hide)
+    )
+    (property "Datasheet" "" (id 3) (at 39.37 120.65 0)
       (effects (font (size 1.27 1.27)) hide)
     )
@@
     (pin "1")
   )
-  (symbol (lib_id "0.power-symbols:GNDD") (at 45.085 120.65 0) (unit 1)
-    (in_bom yes) (on_board yes) (fields_autoplaced)
-    (property "Reference" "#PWR0128" (id 0) (at 45.085 127 0)
-      (effects (font (size 1.27 1.27)) hide)
-    )
-    (property "Value" "GNDD" (id 1) (at 45.085 125.0934 0))
-    (property "Footprint" "" (id 2) (at 45.085 120.65 0)
-      (effects (font (size 1.27 1.27)) hide)
-    )
-    (property "Datasheet" "" (id 3) (at 45.085 120.65 0)
-      (effects (font (size 1.27 1.27)) hide)
-    )
-    (pin "1")
-  )
   (symbol (lib_id "0.power-symbols:+BATT") (at 45.085 50.8 0) (unit 1)
     (in_bom yes) (on_board yes) (fields_autoplaced)
@@
     (pin "1")
   )
-  (symbol (lib_id "0.power-symbols:GNDD") (at 45.085 163.195 0) (unit 1)
-    (in_bom yes) (on_board yes) (fields_autoplaced)
-    (property "Reference" "#PWR0131" (id 0) (at 45.085 169.545 0)
-      (effects (font (size 1.27 1.27)) hide)
-    )
-    (property "Value" "GNDD" (id 1) (at 45.085 167.6384 0))
-    (property "Footprint" "" (id 2) (at 45.085 163.195 0)
-      (effects (font (size 1.27 1.27)) hide)
-    )
-    (property "Datasheet" "" (id 3) (at 45.085 163.195 0)
-      (effects (font (size 1.27 1.27)) hide)
-    )
-    (pin "1")
-  )
   (symbol (lib_id "0.power-symbols:+5V") (at 157.48 172.085 0) (unit 1)
     (in_bom yes) (on_board yes) (fields_autoplaced)
@@
     )
     (property "Datasheet" "" (id 3) (at 32.385 135.255 0)
+      (effects (font (size 1.27 1.27)) hide)
+    )
+    (pin "1")
+  )
+  (symbol (lib_id "0.power-symbols:GND") (at 39.37 163.195 0) (unit 1)
+    (in_bom yes) (on_board yes)
+    (property "Reference" "#PWR054" (id 0) (at 39.37 169.545 0)
+      (effects (font (size 1.27 1.27)) hide)
+    )
+    (property "Value" "GND" (id 1) (at 39.37 167.6384 0))
+    (property "Footprint" "" (id 2) (at 39.37 163.195 0)
+      (effects (font (size 1.27 1.27)) hide)
+    )
+    (property "Datasheet" "" (id 3) (at 39.37 163.195 0)
       (effects (font (size 1.27 1.27)) hide)
     )
@@
     (pin "1")
   )
+  (symbol (lib_id "0.power-symbols:GND") (at 45.085 120.65 0) (unit 1)
+    (in_bom yes) (on_board yes)
+    (property "Reference" "#PWR056" (id 0) (at 45.085 127 0)
+      (effects (font (size 1.27 1.27)) hide)
+    )
+    (property "Value" "GND" (id 1) (at 45.085 125.0934 0))
+    (property "Footprint" "" (id 2) (at 45.085 120.65 0)
+      (effects (font (size 1.27 1.27)) hide)
+    )
+    (property "Datasheet" "" (id 3) (at 45.085 120.65 0)
+      (effects (font (size 1.27 1.27)) hide)
+    )
+    (pin "1")
+  )
   (symbol (lib_name "MPM3610_1") (lib_id "1.semi.ic.pmic.voltagereg:MPM3610") (at 61.595 107.95 0) (unit 1)
     (in_bom yes) (on_board yes) (fields_autoplaced)
@@
     (pin "2")
   )
+  (symbol (lib_id "0.power-symbols:GND") (at 45.085 163.195 0) (unit 1)
+    (in_bom yes) (on_board yes)
+    (property "Reference" "#PWR059" (id 0) (at 45.085 169.545 0)
+      (effects (font (size 1.27 1.27)) hide)
+    )
+    (property "Value" "GND" (id 1) (at 45.085 167.6384 0))
+    (property "Footprint" "" (id 2) (at 45.085 163.195 0)
+      (effects (font (size 1.27 1.27)) hide)
+    )
+    (property "Datasheet" "" (id 3) (at 45.085 163.195 0)
+      (effects (font (size 1.27 1.27)) hide)
+    )
+    (pin "1")
+  )
   (symbol (lib_id "2.passive:R") (at 43.18 98.425 0) (unit 1)
     (in_bom yes) (on_board yes)
@@
     (pin "1")
     (pin "2")
-  )
-  (symbol (lib_id "0.power-symbols:GNDD") (at 39.37 120.65 0) (unit 1)
-    (in_bom yes) (on_board yes) (fields_autoplaced)
-    (property "Reference" "#PWR054" (id 0) (at 39.37 127 0)
-      (effects (font (size 1.27 1.27)) hide)
-    )
-    (property "Value" "GNDD" (id 1) (at 39.37 125.0934 0))
-    (property "Footprint" "" (id 2) (at 39.37 120.65 0)
-      (effects (font (size 1.27 1.27)) hide)
-    )
-    (property "Datasheet" "" (id 3) (at 39.37 120.65 0)
-      (effects (font (size 1.27 1.27)) hide)
-    )
-    (pin "1")
   )
   (symbol (lib_id "0.power-symbols:GND") (at 212.725 120.015 0) (unit 1)
@@
     (pin "2")
   )
-  (symbol (lib_id "0.power-symbols:GNDD") (at 39.37 163.195 0) (unit 1)
-    (in_bom yes) (on_board yes) (fields_autoplaced)
-    (property "Reference" "#PWR056" (id 0) (at 39.37 169.545 0)
-      (effects (font (size 1.27 1.27)) hide)
-    )
-    (property "Value" "GNDD" (id 1) (at 39.37 167.6384 0))
-    (property "Footprint" "" (id 2) (at 39.37 163.195 0)
-      (effects (font (size 1.27 1.27)) hide)
-    )
-    (property "Datasheet" "" (id 3) (at 39.37 163.195 0)
-      (effects (font (size 1.27 1.27)) hide)
-    )
-    (pin "1")
-  )
   (symbol (lib_id "2.passive:C") (at 161.925 107.95 0) (unit 1)

Commit message: updates
Parts:
- added D11, D6: LED, 2_Passives_Resistors_SMD_IPC:R_1608_603_B, symbol 1.semi.opto:LED
- added R16, R58, R59, R60, R61: 300, 2_Passives_Resistors_SMD_IPC:R_1608_603_B, symbol 2.passive:R
Connections:
- net +3V3: no longer R41.1, R42.1, R43.1
- net +5V: no longer R46.1, R47.1
- net 3-3V_2: now also R41.1, R42.1, R43.1
- net 3-3V_3: now also R16.1, R58.1, R59.1
- net 5V_2: now also R46.1, R47.1
- net 5V_3: now also R60.1, R61.1
- net GND: now also D11.1 (K), D6.1 (K); no longer D7.1 (K)
- net GNDD: now also D7.1 (K)
- new net: D6.2 (A), R16.2, R58.2, R59.2
- new net: D11.2 (A), R60.2, R61.2
Other:
- note added: "ADD 12V INDICATOR LIGHTS"
- note removed: "Add 16V 3A"
- note removed: "add 24v 3a"
- note removed: "add 48v 3a"
- moved on the sheet: D10, D7, D8, D9, R38, R39, R40, R41, R42, R43, R44, R45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

Commit message: updates
Parts:
- added C33, C35: 1uF, 2_Passives_Capacitors_SMD_IPC:C_1608_603_B, symbol 2.passive:C
- added C34: 100pF, 2_Passives_Capacitors_SMD_IPC:C_1608_603_B, symbol 2.passive:C
- added C36, C38: 10uF, 2_Passives_Capacitors_SMD_IPC:C_1608_603_B, symbol 2.passive:C
- added C37: 10uF, 2_Passives_Capacitors_SMD_IPC:C_2012_805_B, symbol 2.passive:C
- added D1, D12, D2: D_Schottky, 1_Semi_Discrete_Diodes_SMD:D_SOD-123F, symbol 1.semi.discrete:D_Schottky
- added D13, D14, D15, D16: LED, 1_Semi_Discrete_Diodes_SMD:D_0603, symbol 1.semi.opto:LED
- added R66, R67: 300, 2_Passives_Resistors_SMD_IPC:R_1608_603_B, symbol 2.passive:R
- added R68, R69, R70: 500, 2_Passives_Resistors_SMD_IPC:R_2012_805_B, symbol 2.passive:R
- added U34: AP2213-8_SOIC, 1_Semi_Misc:SOIC-8_3.9x4.9mm_P1.27mm, symbol 1.semi.ic.pmic.voltagereg:AP2213-8_SOIC
- added U36: LM1085-5.0, 1_Semi_TO_SOT:TO-263-3_TabPin2, symbol 1.semi.ic.pmic.voltagereg:LM1085
- D10, D11, D6, D7, D8, D9: footprint 2_Passives_Resistors_SMD_IPC:R_1608_603_B -> 1_Semi_Discrete_Diodes_SMD:D_0603
Connections:
- net +12V: now also R68.2
- net +3V3: now also C35.1, C36.1, U34.3 (VOUT); no longer C14.1, R32.1, R38.1, R39.1, R40.1, U4.9 (OUT)
- net +BATT: now also C37.1, U36.3 (VIN)
- net 12V_2: now also R69.2
- net 12V_3: now also R70.2
- net GND: now also C11.2, C14.2, D7.1 (K), R33.2, U4.14 (PGND), U4.3 (AGND), C37.2, C38.2, D13.1 (K), D14.1 (K), D15.1 (K), D16.1 (K), U36.1 (ADJ)
- net GNDD: now also C33.1, C34.2, C35.2, C36.2, U34.5 (GND), U34.6 (GND), U34.7 (GND), U34.8 (GND); no longer C11.2, C14.2, D7.1 (K), R33.2, U4.14 (PGND), U4.3 (AGND)
- new net: D15.2 (A), R69.1
- new net: D14.2 (A), R68.1
- new net: D13.2 (A), R66.2, R67.2
- new net: C33.2, D1.1 (K), D12.1 (K), D2.1 (K), U34.1 (EN), U34.2 (VIN)
- new net: C34.1, U34.4 (BYP)
- new net: D16.2 (A), R70.1
- new net 3-3V_1: C14.1, R32.1, R38.1, R39.1, R40.1, U4.9 (OUT)
- new net 5V_4: C38.1, R66.1, R67.1, U36.2 (VOUT)
- new net BATT_1_PWR: D2.2 (A)
- new net BATT_2_PWR: D12.2 (A)
- new net VUSB: D1.2 (A)
- no-connect marks 30 -> 18
Other:
- note added: "ADD 12V INDICATOR LIGHTS + and change LED footprints"
- note added: "Dedicated Microprocessor PSU"
- note removed: "ADD 12V INDICATOR LIGHTS"
