File: 1.0/processor.kicad_sch (KiCad schematic)
At the start: 13 parts

Commit message: updates
Parts:
- removed D?: D_Schottky, symbol 1.semi.discrete:D_Schottky
- added C31, C32: 10uF, 2_Passives_Capacitors_SMD_IPC:C_1608_603_B, symbol 2.passive:C
- added D2: D_Schottky, 1_Semi_Discrete_Diodes_SMD:D_SOD-323, symbol 1.semi.discrete:D_Schottky
- added TP10, TP11, TP12, TP2, TP3, TP4, TP5, TP6, TP7, TP8, TP9, TP?: TEST, 0_misc:test_point_2mm_square, symbol 5.connector.interconnect:TEST
- D1: renamed from D?; footprint (none) -> 1_Semi_Discrete_Diodes_SMD:D_SOD-323
- IC1: renamed from IC?; Height 0.8 -> (none); Manufacturer_Name GigaDevice -> (none); Manufacturer_Part_Number GD25Q16CWIGR -> (none); Mouser Part Number 363-GD25Q16CWIGR -> (none); Mouser Price/Stock https://www.mouser.co.uk/ProductDetail/GigaDevice/GD25Q16CW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 -> (none)
- IC2: renamed from IC?; Arrow Part Number ATSAMD21G18A-MUT -> (none); Arrow Price/Stock https://www.arrow.com/en/products/atsamd21g18a-mut/microchi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 -> (none); Height 0.9 -> (none); Manufacturer_Name Microchip -> (none); Manufacturer_Part_Number ATSAMD21G18A-MUT -> (none); Mouser Part Number 556-ATSAMD21G18A-MUT -> (none); Mouser Price/Stock https://www.mouser.co.uk/ProductDetail/Microchip-Technology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 -> (none)
- Q1: renamed from Q?; footprint 1.Semi.TO_SOT:SOT-23 -> 1_Semi_TO_SOT:SOT-23
- R1: renamed from R?; value 10K -> 10k
- R2, R3, R4: renamed from R?; footprint (none) -> 2_Passives_Resistors_SMD_IPC:R_1608_603_B
- SW1: renamed from SW?; footprint (none) -> 3_Electromechanical_Buttons_Switches_SMD:CK_PTS645_SMD
- TP1: renamed from TP?; footprint (none) -> 0_misc:test_point_1.0mm_square
- gave numbers to parts that had none: 2
Connections:
- net BATT_1_CTL: now also TP11.1
- net BATT_1_CURR: now also TP4.1
- net BATT_1_VSENSE: now also TP3.1
- net BATT_2_CTL: now also TP12.1
- net BATT_2_CURR: now also IC2.10 (PA05), TP8.1; no longer IC2.9 (PA04)
- net BATT_2_VSENSE: now also IC2.9 (PA04); no longer IC2.3 (PA02)
- net GND: now also C31.2, C32.2, TP?.1; no longer SW1.2, SW1.4
- net GNDD: now also SW1.3
- net MISO: now also TP9.1
- net MOSI: now also TP5.1
- net RESET: now also R2.2; no longer IC2.40 (~{RESET}), Q1.3 (C), R4.2, SW1.1, SW1.3, TP1.1
- net SCK: now also TP6.1
- net SD_CS: now also TP10.1
- net VIN: now also C31.1, C32.1, D2.1 (K)
- net VUSB: now also D2.2 (A)
- net at Q1.1 (B), R3.1: no longer R2.2
- net A5_SENSE: now reaches IC2.47 (PB02)
- net A5_SENSE: now also TP2.1
- new net A0_SENSE: IC2.3 (PA02), TP7.1
- new net ~{RESET_RAW}: IC2.40 (~{RESET}), Q1.3 (C), R4.2, SW1.1, TP1.1
Other:
- note added: "Breakout TP"
- moved on the sheet: C1, C2, D1, IC1, IC2, Q1, R1, R2, R3, R4, SW1, TP1

Commit message: updates
Parts:
- gave numbers to parts that had none: 1
Changed lines of the file:
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@@
   (symbol (lib_id "5.connector.interconnect:TEST") (at 161.29 167.005 0) (unit 1)
     (in_bom yes) (on_board yes)
-    (property "Reference" "TP?" (id 0) (at 159.385 158.115 0)
+    (property "Reference" "TP13" (id 0) (at 159.385 158.115 0)
       (effects (font (size 1.27 1.27)) (justify left))
     )
@@
   (symbol (lib_id "0.power-symbols:GND") (at 161.29 175.26 0) (unit 1)
     (in_bom yes) (on_board yes) (fields_autoplaced)
-    (property "Reference" "#PWR?" (id 0) (at 161.29 181.61 0)
+    (property "Reference" "#PWR0139" (id 0) (at 161.29 181.61 0)
       (effects (font (size 1.27 1.27)) hide)
     )

Commit message: updates
Parts:
- removed TP2: TEST, 0_misc:test_point_2mm_square, symbol 5.connector.interconnect:TEST
- added TP14, TP15, TP16: TEST, 0_misc:test_point_2mm_square, symbol 5.connector.interconnect:TEST
Connections:
- net A5_SENSE: now also TP15.1
- net BATT_2_CTL: now also TP14.1; no longer TP12.1
- net BATT_2_CURR: now also TP12.1; no longer TP8.1
- net BATT_2_VSENSE: now also TP8.1
- net GND: now also TP16.1; no longer TP13.1
- net GNDD: now also TP13.1
Other:
- moved on the sheet: TP10, TP11, TP13, TP3, TP4, TP5, TP6, TP7, TP9

Commit message: updates
Parts:
- removed D1, D2: D_Schottky, 1_Semi_Discrete_Diodes_SMD:D_SOD-323, symbol 1.semi.discrete:D_Schottky
- IC1: footprint 1_Semi_Misc:PSON50P200X300X50-9N -> 1_Semi_Misc:SOIC-8_3.9x4.9mm_P1.27mm
- SW1: footprint 3_Electromechanical_Buttons_Switches_SMD:CK_PTS645_SMD -> 3_Electromechanical_Buttons_Switches_SMD:KMR243GLFG
Connections:
- net VIN is gone; now on net +3V3: C1.1, C31.1, C32.1, IC2.17 (VDDIO_1), IC2.36 (VDDIO_2), IC2.44 (VDDIN), IC2.6 (VDDANA)
- net BATT_1_CTL: now also IC2.27 (PA18); no longer IC2.26 (PA17)
- net BATT_2_CTL: now also IC2.26 (PA17); no longer IC2.27 (PA18)
- net BATT_2_CURR: now also IC2.9 (PA04); no longer IC2.10 (PA05)
- net BATT_2_VSENSE: now also IC2.10 (PA05); no longer IC2.9 (PA04)
- net GND: no longer C1.2, C31.2, C32.2
- net GNDD: now also C1.2, C31.2, C32.2
Other:
- moved on the sheet: C1, C31, C32, TP10, TP11, TP12, TP13, TP14, TP15, TP16, TP3, TP4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
